Commit message: $user_name param cannot be obtained in xacro.

File: urdf/human/human.urdf.xacro (robot description, xacro)
@@ -1,11 +1,11 @@
 <?xml version="1.0" ?>
 <robot name="human" xmlns:xacro="http://www.ros.org/wiki/xacro">
-  <xacro:include filename="$(find imu_human_pkg)/urdf/macros/measurements.xacro" />
-  <xacro:include filename="$(find imu_human_pkg)/urdf/macros/materials.xacro" />
-  <xacro:include filename="$(find imu_human_pkg)/urdf/macros/human.gazebo.xacro" />
-  <xacro:include filename="$(find imu_human_pkg)/urdf/macros/human.transmission.xacro" />
-  <xacro:include filename="$(find imu_human_pkg)/urdf/macros/spherical.xacro"/>
-  <xacro:include filename="$(find imu_human_pkg)/urdf/human/human_lower.xacro"/>
-  <xacro:include filename="$(find imu_human_pkg)/urdf/human/human_upper.xacro"/>
+  <xacro:include filename="$(find appirh_project_helse_frde)/urdf/macros/measurements.xacro" />
+  <xacro:include filename="$(find appirh_project_helse_frde)/urdf/macros/materials.xacro" />
+  <xacro:include filename="$(find appirh_project_helse_frde)/urdf/macros/human.gazebo.xacro" />
+  <xacro:include filename="$(find appirh_project_helse_frde)/urdf/macros/human.transmission.xacro" />
+  <xacro:include filename="$(find appirh_project_helse_frde)/urdf/macros/spherical.xacro"/>
+  <xacro:include filename="$(find appirh_project_helse_frde)/urdf/human/human_lower.xacro"/>
+  <xacro:include filename="$(find appirh_project_helse_frde)/urdf/human/human_upper.xacro"/>
   <create/>
   <link name="world"/>

File: urdf/macros/measurements.xacro (robot description, xacro)
@@ -1,5 +1,7 @@
 <?xml version="1.0"?>
 <robot name="human" xmlns:xacro="http://www.ros.org/wiki/xacro">
-  <xacro:property name="human_params" value="${load_yaml('$(find imu_human_pkg)/config/human.yaml')}"/>
+  <xacro:property name="user" value="${xacro.load_yaml('$(find appirh_project_helse_frde)/config/user.yaml')}"/>
+  <xacro:property name="user_name" value="${user['user_name']}" />
+  <xacro:property name="human_params" value="${xacro.load_yaml('$(find appirh_project_helse_frde)/test_users/${user_name}/human.yaml')}"/>
   <xacro:property name="l_neck" value="0.053" />
   <xacro:property name="head" value="0.212-${l_neck}" />
