Commit message: cleaned URDFs - no inertia/collision. Rest is backup

File: urdf/human/human_lower.xacro (robot description, xacro)
@@ -3,5 +3,5 @@
     <xacro:macro name="human_lower">
     <joint name="base_to_lower_trunk" type="fixed">
-        <origin rpy="0 0 0" xyz="0 0 ${thickness+l_shank+l_thigh+l_lower_trunk/2}"/>
+        <origin rpy="0 ${-pi/2} 0" xyz="0 0 ${thickness+l_shank+l_thigh+l_lower_trunk/2}"/>
         <parent link="human_base_link"/>
         <child link="lower_trunk"/>
@@ -87,5 +87,5 @@
     </link>
     <joint name="right_thight_to_shank" type="fixed">
-        <origin rpy="0 0 0" xyz="0 0 ${-l_thigh}"/>
+        <origin rpy="0 ${pi/2} 0" xyz="0 0 ${-l_thigh}"/>
         <parent link="right_thigh"/>
         <child link="right_shank"/>
@@ -143,5 +143,5 @@
     </link>
         <joint name="left_thight_to_shank" type="fixed">
-        <origin rpy="0 0 0" xyz="0 0 ${-l_thigh}"/>
+        <origin rpy="0 ${pi/2} 0" xyz="0 0 ${-l_thigh}"/>
         <parent link="left_thigh"/>
         <child link="left_shank"/>

File: urdf/macros/measurements.xacro (robot description, xacro)
@@ -16,15 +16,15 @@
   <xacro:property name="l_foot" value="${w_foot*4}" />
   <xacro:property name="whole_body" value="1.7268" />
-  <xacro:property name="thickness" value="0.02" />
+  <xacro:property name="thickness" value="0.04" />
   <xacro:property name="r_neck" value="${l_neck/1.5}" />
   <xacro:property name="r_head" value="0.15" />
-  <xacro:property name="r_upper_trunk" value="${l_upper_trunk/2}" />
-  <xacro:property name="r_lower_trunk" value="${l_lower_trunk}" />
-  <xacro:property name="r_upper_arm" value="${l_upper_arm/6.5}" />
-  <xacro:property name="r_forearm" value="${l_forearm/7}" />
-  <xacro:property name="w_hand" value="${l_hand/4}" />
-  <xacro:property name="r_thigh" value="${l_thigh/4.5}" />
-  <xacro:property name="r_shank" value="${l_shank/5.5}" />
-  <xacro:property name="w_foot" value="0.06" />
+  <xacro:property name="r_upper_trunk" value="${l_upper_trunk/1.3}" />
+  <xacro:property name="r_lower_trunk" value="${r_upper_trunk/2}" />
+  <xacro:property name="r_upper_arm" value="${thickness}"  />
+  <xacro:property name="r_forearm" value="${thickness}" />
+  <xacro:property name="w_hand" value="${2*thickness}" />
+  <xacro:property name="r_thigh" value="${thickness}" />
+  <xacro:property name="r_shank" value="${thickness}" />
+  <xacro:property name="w_foot" value="${2*thickness}" />
   <xacro:property name="cm_head" value="0.361" />
   <xacro:property name="cm_upper_trunk" value="0.497" />
@@ -46,7 +46,9 @@
   <xacro:property name="d_shank" value="1100.2" />
   <xacro:property name="d_foot" value="1089.3" />
+  <xacro:property name="r_base_link" value="0.01" />
+  <xacro:property name="unit_scale" value="0.0001" />
   <!-- <xacro:property name="mass" value="${pi*l_upper_arm*pow(w_upper_arm,2)*d_upper_arm*0.001}" />
   <xacro:property name="radius" value="0.1" /> -->
-  <xacro:property name="m_base_link" value="0.01" />
+  <!-- <xacro:property name="m_base_link" value="0.01" />
   <xacro:property name="r_base_link" value="0.01" />
   <xacro:property name="unit_scale" value="0.0001" />
@@ -60,4 +62,4 @@
   <xacro:property name="m_shank" value="${pi*l_shank*pow(r_shank,2)*d_shank*unit_scale}" />
   <xacro:property name="m_hand" value="${l_hand*w_hand*thickness*d_hand*unit_scale}" />
-  <xacro:property name="m_foot" value="${l_foot*w_foot*thickness*d_foot*unit_scale}" />
+  <xacro:property name="m_foot" value="${l_foot*w_foot*thickness*d_foot*unit_scale}" />  -->
 </robot>
