Commit message: some more dummy ui for new user and progress windows

File: urdf/macros/measurements.xacro (robot description, xacro)
@@ -3,5 +3,6 @@
   <xacro:property name="user" value="${xacro.load_yaml('$(find appirh_project_helse_frde)/config/user.yaml')}"/>
   <xacro:property name="user_name" value="${user['user_name']}" />
-  <xacro:property name="human_params" value="${xacro.load_yaml('$(find appirh_project_helse_frde)/test_users/${user_name}/human.yaml')}"/>
+  <!--<xacro:property name="human_params" value="${xacro.load_yaml('$(find appirh_project_helse_frde)/test_users/${user_name}/human.yaml')}"/>-->
+  <xacro:property name="human_params" value="${xacro.load_yaml('/home/gizem/catkin_ws/src/appirh_project_helse_frde/test_users/${user_name}/human.yaml')}"/>
   <xacro:property name="l_neck" value="0.053" />
   <xacro:property name="head" value="0.212-${l_neck}" />

Commit message: found a way to easily switch patients

File: urdf/macros/measurements.xacro (robot description, xacro)
@@ -1,8 +1,5 @@
 <?xml version="1.0"?>
 <robot name="human" xmlns:xacro="http://www.ros.org/wiki/xacro">
-  <xacro:property name="user" value="${xacro.load_yaml('$(find appirh_project_helse_frde)/config/user.yaml')}"/>
-  <xacro:property name="user_name" value="${user['user_name']}" />
-  <!--<xacro:property name="human_params" value="${xacro.load_yaml('$(find appirh_project_helse_frde)/test_users/${user_name}/human.yaml')}"/>-->
-  <xacro:property name="human_params" value="${xacro.load_yaml('/home/gizem/catkin_ws/src/appirh_project_helse_frde/test_users/${user_name}/human.yaml')}"/>
+  <xacro:property name="human_params" value="${xacro.load_yaml('$(find appirh_project_helse_frde)/dynamic_patient_files/human.yaml')}"/>
   <xacro:property name="l_neck" value="0.053" />
   <xacro:property name="head" value="0.212-${l_neck}" />
