Commit message: backup round parts

File: urdf/human-stick-figure/human_upper.xacro (robot description, xacro)
@@ -14,4 +14,32 @@
         </visual>
     </link>
+    <link name="round_up_upper_trunk">
+        <visual>
+        <origin rpy="0 0 0" xyz="0 0 0"/>
+        <geometry>
+            <cylinder length="${r_upper_trunk}" radius="${thickness}"/>
+        </geometry>
+        <material name="orange"/>
+        </visual>
+    </link>
+    <joint name="upper_round_fixed_joint" type="fixed">
+        <origin xyz="0 0 ${l_upper_trunk}" rpy="${-pi/2} 0 0" />
+        <parent link="upper_trunk"/>
+        <child link="round_up_upper_trunk"/>
+    </joint>
+    <link name="round_left_upper_trunk">
+        <visual>
+        <origin rpy="0 0 0" xyz="0 0 0"/>
+        <geometry>
+            <cylinder length="${l_upper_trunk}" radius="${thickness}"/>
+        </geometry>
+        <material name="green"/>
+        </visual>
+    </link>
+    <joint name="left_round_fixed_joint" type="fixed">
+        <origin xyz="0 ${-r_upper_trunk/2} ${l_upper_trunk/2}" rpy="0 0 0" />
+        <parent link="upper_trunk"/>
+        <child link="round_left_upper_trunk"/>
+    </joint>
     <xacro:spherical name="right_shoulder" parent="upper_trunk" child="right_upper_arm" x="1" y="1" z="1">
         <origin rpy="0 0 0" xyz="0 ${-r_upper_trunk} ${l_upper_trunk}"/>

Commit message: head mesh looks like fine

File: urdf/human-stick-figure/human_upper.xacro (robot description, xacro)
@@ -14,32 +14,4 @@
         </visual>
     </link>
-    <link name="round_up_upper_trunk">
-        <visual>
-        <origin rpy="0 0 0" xyz="0 0 0"/>
-        <geometry>
-            <cylinder length="${r_upper_trunk}" radius="${thickness}"/>
-        </geometry>
-        <material name="orange"/>
-        </visual>
-    </link>
-    <joint name="upper_round_fixed_joint" type="fixed">
-        <origin xyz="0 0 ${l_upper_trunk}" rpy="${-pi/2} 0 0" />
-        <parent link="upper_trunk"/>
-        <child link="round_up_upper_trunk"/>
-    </joint>
-    <link name="round_left_upper_trunk">
-        <visual>
-        <origin rpy="0 0 0" xyz="0 0 0"/>
-        <geometry>
-            <cylinder length="${l_upper_trunk}" radius="${thickness}"/>
-        </geometry>
-        <material name="green"/>
-        </visual>
-    </link>
-    <joint name="left_round_fixed_joint" type="fixed">
-        <origin xyz="0 ${-r_upper_trunk/2} ${l_upper_trunk/2}" rpy="0 0 0" />
-        <parent link="upper_trunk"/>
-        <child link="round_left_upper_trunk"/>
-    </joint>
     <xacro:spherical name="right_shoulder" parent="upper_trunk" child="right_upper_arm" x="1" y="1" z="1">
         <origin rpy="0 0 0" xyz="0 ${-r_upper_trunk} ${l_upper_trunk}"/>
@@ -111,9 +83,10 @@
     <link name="head">
         <visual>
-        <origin rpy="0 0 0" xyz="0 0 ${r_head}"/>
+        <origin rpy="${pi/2} 0 ${pi/2}" xyz="${r_head/4} 0 ${1.5*r_head}"/>
         <geometry>
-            <sphere radius="${r_head}"/>
+            <!-- <sphere radius="${r_head}"/> -->
+            <mesh filename="file://$(arg meshDirectory)headMesh.obj" scale=".12 .12 .08"/>
         </geometry>
-        <material name="white"/>
+        <material name="orange"/>
         </visual>
     </link>
@@ -149,4 +122,47 @@
         </visual>
     </link>
+    <!-- Fixed visual links and joints: -->
+    <link name="round_up_upper_trunk">
+        <visual>
+        <origin rpy="0 0 0" xyz="0 0 0"/>
+        <geometry>
+            <cylinder length="${r_upper_trunk}" radius="${thickness}"/>
+        </geometry>
+        <material name="orange"/>
+        </visual>
+    </link>
+    <joint name="upper_round_fixed_joint" type="fixed">
+        <origin xyz="0 0 ${l_upper_trunk}" rpy="${-pi/2} 0 0" />
+        <parent link="upper_trunk"/>
+        <child link="round_up_upper_trunk"/>
+    </joint>
+    <link name="round_left_upper_trunk">
+        <visual>
+        <origin rpy="0 0 0" xyz="0 0 0"/>
+        <geometry>
+            <cylinder length="${l_upper_trunk}" radius="${thickness}"/>
+        </geometry>
+        <material name="orange"/>
+        </visual>
+    </link>
+    <joint name="left_round_fixed_joint" type="fixed">
+        <origin xyz="0 ${r_upper_trunk/2} ${l_upper_trunk/2}" rpy="0 0 0" />
+        <parent link="upper_trunk"/>
+        <child link="round_left_upper_trunk"/>
+    </joint>
+    <link name="round_right_upper_trunk">
+        <visual>
+        <origin rpy="0 0 0" xyz="0 0 0"/>
+        <geometry>
+            <cylinder length="${l_upper_trunk}" radius="${thickness}"/>
+        </geometry>
+        <material name="orange"/>
+        </visual>
+    </link>
+    <joint name="right_round_fixed_joint" type="fixed">
+        <origin xyz="0 ${-r_upper_trunk/2} ${l_upper_trunk/2}" rpy="0 0 0" />
+        <parent link="upper_trunk"/>
+        <child link="round_right_upper_trunk"/>
+    </joint>
 </xacro:macro>
 </robot>

File: urdf/macros/materials.xacro (robot description, xacro)
@@ -14,5 +14,5 @@
   </material>
   <material name="orange">
-    <color rgba="1 0.6 0 0.8"/>
+    <color rgba="1 0.6 0 1"/>
   </material>
 </robot>

File: urdf/macros/measurements.xacro (robot description, xacro)
@@ -16,15 +16,15 @@
   <xacro:property name="l_foot" value="${w_foot*4}" />
   <xacro:property name="whole_body" value="1.7268" />
-  <xacro:property name="thickness" value="0.04" />
+  <xacro:property name="thickness" value="0.07" />
   <xacro:property name="r_neck" value="${l_neck/1.5}" />
   <xacro:property name="r_head" value="0.15" />
-  <xacro:property name="r_upper_trunk" value="${l_upper_trunk/1.3}" />
+  <xacro:property name="r_upper_trunk" value="${l_upper_trunk/1.8}" />
   <xacro:property name="r_lower_trunk" value="${r_upper_trunk/2}" />
-  <xacro:property name="r_upper_arm" value="${thickness}"  />
-  <xacro:property name="r_forearm" value="${thickness}" />
-  <xacro:property name="w_hand" value="${2*thickness}" />
-  <xacro:property name="r_thigh" value="${thickness}" />
-  <xacro:property name="r_shank" value="${thickness}" />
-  <xacro:property name="w_foot" value="${2*thickness}" />
+  <xacro:property name="r_upper_arm" value="${thickness/2}"  />
+  <xacro:property name="r_forearm" value="${thickness/2}" />
+  <xacro:property name="w_hand" value="${thickness}" />
+  <xacro:property name="r_thigh" value="${thickness/2}" />
+  <xacro:property name="r_shank" value="${thickness/2}" />
+  <xacro:property name="w_foot" value="${thickness}" />
   <xacro:property name="cm_head" value="0.361" />
   <xacro:property name="cm_upper_trunk" value="0.497" />
