Commit message: human is done-ish. trying to add chair.

File: urdf/human-stick-figure/human.urdf.xacro (robot description, xacro)
@@ -8,4 +8,5 @@
   <xacro:include filename="$(find appirh_project_helse_frde)/urdf/human-stick-figure/human_lower.xacro"/>
   <xacro:include filename="$(find appirh_project_helse_frde)/urdf/human-stick-figure/human_upper.xacro"/>
+  <xacro:include filename="$(find appirh_project_helse_frde)/urdf/human-stick-figure/objects.xacro"/>
   <create/>
   <link name="world"/>
@@ -28,3 +29,4 @@
   <xacro:human_lower/>
   <xacro:human_upper/>
+  <xacro:objects/>
 </robot>

File: urdf/human-stick-figure/human_lower.xacro (robot description, xacro)
@@ -3,5 +3,5 @@
     <xacro:macro name="human_lower">
     <joint name="base_to_lower_trunk" type="fixed">
-        <origin rpy="0 ${-pi/2} 0" xyz="0 0 ${thickness+l_shank+l_thigh+l_lower_trunk/2}"/>
+        <origin rpy="0 ${-pi/2} 0" xyz="${-l_lower_trunk/2} 0 ${2*l_upper_trunk+r_lower_trunk}"/>
         <parent link="human_base_link"/>
         <child link="lower_trunk"/>

File: urdf/human-stick-figure/human_upper.xacro (robot description, xacro)
@@ -15,5 +15,5 @@
     </link>
     <xacro:spherical name="right_shoulder" parent="upper_trunk" child="right_upper_arm" x="1" y="1" z="1">
-        <origin rpy="0 0 0" xyz="0 ${-r_upper_trunk} ${l_upper_trunk}"/>
+        <origin rpy="0 0 0" xyz="0 ${-r_upper_trunk/1.5} ${l_upper_trunk}"/>
     </xacro:spherical>
     <link name="right_upper_arm">
@@ -27,5 +27,5 @@
     </link>
     <xacro:spherical name="left_shoulder" parent="upper_trunk" child="left_upper_arm" x="-1" y="1" z="-1">
-        <origin rpy="0 0 0" xyz="0 ${r_upper_trunk} ${l_upper_trunk}"/>
+        <origin rpy="0 0 0" xyz="0 ${r_upper_trunk/1.5} ${l_upper_trunk}"/>
     </xacro:spherical>
     <link name="left_upper_arm">
@@ -98,5 +98,5 @@
     <link name="right_hand">
         <visual>
-        <origin rpy="${-pi/2} ${pi/2} 0" xyz="0 0 ${-l_hand/2}"/>
+        <origin rpy="${-pi/2} ${pi/2} 0" xyz="0 0 ${-w_hand/2}"/>
         <geometry>
             <sphere radius="${w_hand}"/>
@@ -115,5 +115,5 @@
     <link name="left_hand">
         <visual>
-        <origin rpy="${pi/2} ${pi/2} 0" xyz="0 0 ${-l_hand/2}"/>
+        <origin rpy="${pi/2} ${pi/2} 0" xyz="0 0 ${-w_hand/2}"/>
         <geometry>
             <sphere radius="${w_foot}"/>
@@ -165,4 +165,60 @@
         <child link="round_right_upper_trunk"/>
     </joint>
+    <link name="ballup_round_right_upper_trunk">
+        <visual>
+        <origin rpy="0 0 0" xyz="0 0 0"/>
+        <geometry>
+            <sphere radius="${thickness}"/>
+        </geometry>
+        <material name="orange"/>
+        </visual>
+    </link>
+    <joint name="round_right_upper_trunk" type="fixed">
+        <origin xyz="0 ${-r_upper_trunk/1.5} ${l_upper_trunk}" rpy="0 0 0" />
+        <parent link="upper_trunk"/>
+        <child link="ballup_round_right_upper_trunk"/>
+    </joint>
+    <link name="ballup_round_left_upper_trunk">
+        <visual>
+        <origin rpy="0 0 0" xyz="0 0 0"/>
+        <geometry>
+            <sphere radius="${thickness}"/>
+        </geometry>
+        <material name="orange"/>
+        </visual>
+    </link>
+    <joint name="round_left_upper_trunk" type="fixed"> <!-- #TODO: Equalize later 1.5 multiplier-->
+        <origin xyz="0 ${r_upper_trunk/1.5} ${l_upper_trunk}" rpy="0 0 0" />
+        <parent link="upper_trunk"/>
+        <child link="ballup_round_left_upper_trunk"/>
+    </joint>
+    <link name="ball_left_elbow">
+        <visual>
+        <origin rpy="0 0 0" xyz="0 0 0"/>
+        <geometry>
+            <sphere radius="${thickness}"/>
+        </geometry>
+        <material name="orange"/>
+        </visual>
+    </link>
+    <joint name="ball_left_elbow" type="fixed">
+        <origin xyz="0 0 ${-l_upper_arm}" rpy="0 0 0" />
+        <parent link="left_upper_arm"/>
+        <child link="ball_left_elbow"/>
+    </joint>
+    <link name="ball_right_elbow">
+        <visual>
+        <origin rpy="0 0 0" xyz="0 0 0"/>
+        <geometry>
+            <sphere radius="${thickness}"/>
+        </geometry>
+        <material name="orange"/>
+        </visual>
+    </link>
+    <joint name="ball_right_elbow" type="fixed">
+        <origin xyz="0 0 ${-l_upper_arm}" rpy="0 0 0" />
+        <parent link="right_upper_arm"/>
+        <child link="ball_right_elbow"/>
+    </joint>
 </xacro:macro>
 </robot>

Commit message: chair with stl

File: urdf/human-stick-figure/human.urdf.xacro (robot description, xacro)
@@ -13,5 +13,5 @@
   <joint name="world_joint" type="fixed">
     <!-- <origin xyz="0 0 0" rpy="0 0 ${pi/2}" /> -->
-    <origin xyz="0 0 0" rpy="0 0 0" />
+    <origin xyz="0 0 -0.55 " rpy="0 0 0" />
     <parent link="world"/>
     <child link="human_base_link"/>
@@ -20,5 +20,5 @@
   <link name="human_base_link">
     <visual>
-    <origin rpy="0 0 0" xyz="0 0 ${thickness+l_shank+l_thigh+l_lower_trunk/2}"/>
+    <origin rpy="0 0 0" xyz="0 0 0"/>
       <geometry>
         <sphere radius="${r_base_link}"/>

File: urdf/human-stick-figure/objects.xacro (robot description, xacro)
@@ -3,6 +3,6 @@
     <xacro:macro name="objects">
     <joint name="base_to_chair_joint" type="fixed">
-        <origin rpy="0 ${-pi/2} 0" xyz="${-l_lower_trunk/2} 0 ${2*l_upper_trunk+r_lower_trunk}"/>
-        <parent link="human_base_link"/>
+        <origin rpy="0 0 ${pi/2}" xyz="${-l_lower_trunk/2} 0 0"/>
+        <parent link="world"/>
         <child link="chair"/>
     </joint>
@@ -11,17 +11,9 @@
             <origin rpy="1.57 0 0" xyz="0 0 0" />
             <geometry>
-                <!-- <mesh filename="chair.obj" /> -->
-                <box size="0.717032 1.000000 0.683208" />
+                <mesh filename="file://$(arg meshDirectory)chair.stl" />
+                <!-- <box size="0.717032 1.000000 0.683208" /> -->
             </geometry>
+            <material name="brown"/>
         </visual>
-        <collision>
-            <geometry>
-                <box size="0.717032 1.000000 0.683208" />
-            </geometry>
-        </collision>
-        <inertial>
-            <mass value="0.0" />
-            <inertia ixx="0.0" ixy="0.0" ixz="0.0" iyy="0.0" iyz="0.0" izz="0.0" />
-        </inertial>
     </link>
     </xacro:macro>

File: urdf/macros/materials.xacro (robot description, xacro)
@@ -16,3 +16,6 @@
     <color rgba="1 0.6 0 1"/>
   </material>
+  <material name="brown">
+    <color rgba="0.54 0.27 0.07 1"/>
+  </material>
 </robot>
